File: project-nrf-C12880MA-motherboard.sch (KiCad schematic (older format))
At the start: 22 parts, among them J1 Left, J2 Right, J3 PJ-036AH-SMT-TR, J4 SM04B-SRSS-TB(LF)(SN), J5 SM04B-SRSS-TB(LF)(SN), J6 SM04B-SRSS-TB(LF)(SN), J7 1702473, J8 C12880MA Breakboard v2, U1 ADS1219IPWR, U2 TPS7A0350PDBVR, U3 LSF0204DPWR

Commit message: First placement
Parts:
- added H? (x4): MountingHole_Pad, MountingHole:MountingHole_2.7mm_M2.5_Pad_Via, symbol Mechanical:MountingHole_Pad
Connections:
- net GND: now also H?.1, H?.1, H?.1, H?.1
Other:
- note added: "Mounting Holes"
- moved on the sheet: J7, R1, S1
Changed lines of the file:
@@
 L power:GND #PWR0104
 U 1 1 6234D28E
-P 9600 2950
-F 0 "#PWR0104" H 9600 2700 50  0001 C CNN
-F 1 "GND" H 9605 2777 50  0000 C CNN
-F 2 "" H 9600 2950 50  0001 C CNN
-F 3 "" H 9600 2950 50  0001 C CNN
-	1    9600 2950
-	1    0    0    -1
-$EndComp
-Text Label 7950 2800 0    50   ~ 0
+P 9050 2950
+F 0 "#PWR0104" H 9050 2700 50  0001 C CNN
+F 1 "GND" H 9055 2777 50  0000 C CNN
+F 2 "" H 9050 2950 50  0001 C CNN
+F 3 "" H 9050 2950 50  0001 C CNN
+	1    9050 2950
+	1    0    0    -1
+$EndComp
+Text Label 7400 2800 0    50   ~ 0
 BUTTON
 $Comp
 L Device:R_Small R1
 U 1 1 62359C57
-P 8350 2550
-F 0 "R1" H 8409 2596 50  0000 L CNN
-F 1 "R_Small" H 8409 2505 50  0000 L CNN
-F 2 "Resistor_SMD:R_0603_1608Metric" H 8350 2550 50  0001 C CNN
-F 3 "~" H 8350 2550 50  0001 C CNN
-	1    8350 2550
+P 7800 2550
+F 0 "R1" H 7859 2596 50  0000 L CNN
+F 1 "R_Small" H 7859 2505 50  0000 L CNN
+F 2 "Resistor_SMD:R_0603_1608Metric" H 7800 2550 50  0001 C CNN
+F 3 "~" H 7800 2550 50  0001 C CNN
+	1    7800 2550
 	1    0    0    -1
 $EndComp
@@
 L B3FS-1010P:B3FS-1010P S1
 U 1 1 6236F713
-P 9050 2800
-F 0 "S1" H 9050 3049 50  0000 C CNN
-F 1 "B3FS-1010P" H 9050 2958 50  0001 C CNN
-F 2 "B3FS-1010:SW_B3FS-1010P" H 9050 2800 50  0001 L BNN
-F 3 "" H 9050 2800 50  0001 L BNN
-F 4 "Compliant" H 9050 2800 50  0001 L BNN "EU_RoHS_Compliance"
-F 5 "B3FS-1010P" H 9050 2800 50  0001 L BNN "Comment"
-	1    9050 2800
-	1    0    0    -1
-$EndComp
-Wire Wire Line
-	9350 2800 9600 2800
-Wire Wire Line
-	7950 2800 8350 2800
-Wire Wire Line
-	8350 2650 8350 2800
-Connection ~ 8350 2800
-Wire Wire Line
-	8350 2800 8750 2800
-Wire Wire Line
-	9600 2800 9600 2950
+P 8500 2800
+F 0 "S1" H 8500 3049 50  0000 C CNN
+F 1 "B3FS-1010P" H 8500 2958 50  0001 C CNN
+F 2 "B3FS-1010:SW_B3FS-1010P" H 8500 2800 50  0001 L BNN
+F 3 "" H 8500 2800 50  0001 L BNN
+F 4 "Compliant" H 8500 2800 50  0001 L BNN "EU_RoHS_Compliance"
+F 5 "B3FS-1010P" H 8500 2800 50  0001 L BNN "Comment"
+	1    8500 2800
+	1    0    0    -1
+$EndComp
+Wire Wire Line
+	8800 2800 9050 2800
+Wire Wire Line
+	7400 2800 7800 2800
+Wire Wire Line
+	7800 2650 7800 2800
+Connection ~ 7800 2800
+Wire Wire Line
+	7800 2800 8200 2800
+Wire Wire Line
+	9050 2800 9050 2950
 $Comp
 L power:+5V #PWR010
@@
 $EndComp
 Wire Wire Line
-	8350 2400 8350 2450
+	7800 2400 7800 2450
 $Comp
 L TPS7A0233PDBVR:TPS7A0233PDBVR U2
@@
 L power:VDD #PWR027
 U 1 1 6257331C
-P 8350 2400
-F 0 "#PWR027" H 8350 2250 50  0001 C CNN
-F 1 "VDD" H 8365 2573 50  0000 C CNN
-F 2 "" H 8350 2400 50  0001 C CNN
-F 3 "" H 8350 2400 50  0001 C CNN
-	1    8350 2400
+P 7800 2400
+F 0 "#PWR027" H 7800 2250 50  0001 C CNN
+F 1 "VDD" H 7815 2573 50  0000 C CNN
+F 2 "" H 7800 2400 50  0001 C CNN
+F 3 "" H 7800 2400 50  0001 C CNN
+	1    7800 2400
 	1    0    0    -1
 $EndComp
@@
 L 1702473:1702473 J7
 U 1 1 62584EF1
-P 8850 3350
-F 0 "J7" H 9080 3396 50  0000 L CNN
-F 1 "1702473" H 9080 3305 50  0000 L CNN
-F 2 "PHOENIX_1702473" H 8850 3350 50  0001 L BNN
-F 3 "" H 8850 3350 50  0001 L BNN
-F 4 "Manufacturer Recommendations" H 8850 3350 50  0001 L BNN "STANDARD"
-F 5 "Phoenix Contact" H 8850 3350 50  0001 L BNN "MANUFACTURER"
-F 6 "MAR20,2012" H 8850 3350 50  0001 L BNN "PARTREV"
-	1    8850 3350
+P 8300 3350
+F 0 "J7" H 8530 3396 50  0000 L CNN
+F 1 "1702473" H 8530 3305 50  0000 L CNN
+F 2 "PHOENIX_1702473" H 8300 3350 50  0001 L BNN
+F 3 "" H 8300 3350 50  0001 L BNN
+F 4 "Manufacturer Recommendations" H 8300 3350 50  0001 L BNN "STANDARD"
+F 5 "Phoenix Contact" H 8300 3350 50  0001 L BNN "MANUFACTURER"
+F 6 "MAR20,2012" H 8300 3350 50  0001 L BNN "PARTREV"
+	1    8300 3350
 	1    0    0    -1
 $EndComp
@@
 $EndComp
 Wire Wire Line
-	8450 3150 8350 3150
-Wire Wire Line
-	8350 3150 8350 2800
+	7900 3150 7800 3150
+Wire Wire Line
+	7800 3150 7800 2800
 $Comp
 L power:GND #PWR028
 U 1 1 625F1955
-P 8350 3650
-F 0 "#PWR028" H 8350 3400 50  0001 C CNN
-F 1 "GND" H 8355 3477 50  0000 C CNN
-F 2 "" H 8350 3650 50  0001 C CNN
-F 3 "" H 8350 3650 50  0001 C CNN
-	1    8350 3650
-	1    0    0    -1
-$EndComp
-Wire Wire Line
-	8450 3550 8350 3550
-Wire Wire Line
-	8350 3550 8350 3650
-Wire Wire Line
-	8450 3250 8350 3250
-Wire Wire Line
-	8350 3250 8350 3550
-Connection ~ 8350 3550
+P 7800 3650
+F 0 "#PWR028" H 7800 3400 50  0001 C CNN
+F 1 "GND" H 7805 3477 50  0000 C CNN
+F 2 "" H 7800 3650 50  0001 C CNN
+F 3 "" H 7800 3650 50  0001 C CNN
+	1    7800 3650
+	1    0    0    -1
+$EndComp
+Wire Wire Line
+	7900 3550 7800 3550
+Wire Wire Line
+	7800 3550 7800 3650
+Wire Wire Line
+	7900 3250 7800 3250
+Wire Wire Line
+	7800 3250 7800 3550
+Connection ~ 7800 3550
 $Comp
 L Device:C_Small C6
@@
 NoConn ~ 1100 2950
 Wire Notes Line
-	500  2050 11200 2050
-Wire Notes Line
 	500  3950 11200 3950
 Wire Notes Line
@@
 Text Label 1250 5450 0    50   ~ 0
 VIDEO
+$Comp
+L Mechanical:MountingHole_Pad H?
+U 1 1 62DE7F5A
+P 10800 2800
+F 0 "H?" H 10900 2803 50  0000 L CNN
+F 1 "MountingHole_Pad" H 10900 2758 50  0001 L CNN
+F 2 "MountingHole:MountingHole_2.7mm_M2.5_Pad_Via" H 10800 2800 50  0001 C CNN
+F 3 "~" H 10800 2800 50  0001 C CNN
+	1    10800 2800
+	1    0    0    -1
+$EndComp
+$Comp
+L Mechanical:MountingHole_Pad H?
+U 1 1 62DE790A
+P 10500 2800
+F 0 "H?" H 10600 2803 50  0000 L CNN
+F 1 "MountingHole_Pad" H 10600 2758 50  0001 L CNN
+F 2 "MountingHole:MountingHole_2.7mm_M2.5_Pad_Via" H 10500 2800 50  0001 C CNN
+F 3 "~" H 10500 2800 50  0001 C CNN
+	1    10500 2800
+	1    0    0    -1
+$EndComp
+$Comp
+L Mechanical:MountingHole_Pad H?
+U 1 1 62DE712E
+P 10200 2800
+F 0 "H?" H 10300 2803 50  0000 L CNN
+F 1 "MountingHole_Pad" H 10300 2758 50  0001 L CNN
+F 2 "MountingHole:MountingHole_2.7mm_M2.5_Pad_Via" H 10200 2800 50  0001 C CNN
+F 3 "~" H 10200 2800 50  0001 C CNN
+	1    10200 2800
+	1    0    0    -1
+$EndComp
+$Comp
+L Mechanical:MountingHole_Pad H?
+U 1 1 62DE5DC9
+P 9900 2800
+F 0 "H?" H 10000 2803 50  0000 L CNN
+F 1 "MountingHole_Pad" H 10000 2758 50  0001 L CNN
+F 2 "MountingHole:MountingHole_2.7mm_M2.5_Pad_Via" H 9900 2800 50  0001 C CNN
+F 3 "~" H 9900 2800 50  0001 C CNN
+	1    9900 2800
+	1    0    0    -1
+$EndComp
+$Comp
+L power:GND #PWR?
+U 1 1 62DF80EC
+P 9900 3000
+F 0 "#PWR?" H 9900 2750 50  0001 C CNN
+F 1 "GND" H 9905 2827 50  0000 C CNN
+F 2 "" H 9900 3000 50  0001 C CNN
+F 3 "" H 9900 3000 50  0001 C CNN
+	1    9900 3000
+	1    0    0    -1
+$EndComp
+Wire Wire Line
+	9900 2900 9900 2950
+Wire Wire Line
+	9900 2950 10200 2950
+Wire Wire Line
+	10200 2950 10200 2900
+Connection ~ 9900 2950
+Wire Wire Line
+	9900 2950 9900 3000
+Wire Wire Line
+	10500 2900 10500 2950
+Wire Wire Line
+	10500 2950 10200 2950
+Connection ~ 10200 2950
+Wire Wire Line
+	10800 2900 10800 2950
+Wire Wire Line
+	10800 2950 10500 2950
+Connection ~ 10500 2950
+Wire Notes Line
+	500  2050 11200 2050
+Wire Notes Line
+	9450 2050 9450 3950
+Text Notes 9550 2250 0    50   ~ 0
+Mounting Holes
 $EndSCHEMATC

Commit message: Placement 2
Parts:
- gave numbers to parts that had none: 4
Other:
- moved on the sheet: H1, H2, H3, H4
Changed lines of the file:
@@
 VIDEO
 $Comp
-L Mechanical:MountingHole_Pad H?
+L Mechanical:MountingHole_Pad H4
 U 1 1 62DE7F5A
-P 10800 2800
-F 0 "H?" H 10900 2803 50  0000 L CNN
-F 1 "MountingHole_Pad" H 10900 2758 50  0001 L CNN
-F 2 "MountingHole:MountingHole_2.7mm_M2.5_Pad_Via" H 10800 2800 50  0001 C CNN
-F 3 "~" H 10800 2800 50  0001 C CNN
-	1    10800 2800
+P 10750 2850
+F 0 "H4" H 10850 2853 50  0000 L CNN
+F 1 "MountingHole_Pad" H 10850 2808 50  0001 L CNN
+F 2 "MountingHole:MountingHole_2.7mm_M2.5_Pad_Via" H 10750 2850 50  0001 C CNN
+F 3 "~" H 10750 2850 50  0001 C CNN
+	1    10750 2850
 	1    0    0    -1
 $EndComp
 $Comp
-L Mechanical:MountingHole_Pad H?
+L Mechanical:MountingHole_Pad H3
 U 1 1 62DE790A
-P 10500 2800
-F 0 "H?" H 10600 2803 50  0000 L CNN
-F 1 "MountingHole_Pad" H 10600 2758 50  0001 L CNN
-F 2 "MountingHole:MountingHole_2.7mm_M2.5_Pad_Via" H 10500 2800 50  0001 C CNN
-F 3 "~" H 10500 2800 50  0001 C CNN
-	1    10500 2800
+P 10450 2850
+F 0 "H3" H 10550 2853 50  0000 L CNN
+F 1 "MountingHole_Pad" H 10550 2808 50  0001 L CNN
+F 2 "MountingHole:MountingHole_2.7mm_M2.5_Pad_Via" H 10450 2850 50  0001 C CNN
+F 3 "~" H 10450 2850 50  0001 C CNN
+	1    10450 2850
 	1    0    0    -1
 $EndComp
 $Comp
-L Mechanical:MountingHole_Pad H?
+L Mechanical:MountingHole_Pad H2
 U 1 1 62DE712E
-P 10200 2800
-F 0 "H?" H 10300 2803 50  0000 L CNN
-F 1 "MountingHole_Pad" H 10300 2758 50  0001 L CNN
-F 2 "MountingHole:MountingHole_2.7mm_M2.5_Pad_Via" H 10200 2800 50  0001 C CNN
-F 3 "~" H 10200 2800 50  0001 C CNN
-	1    10200 2800
+P 10150 2850
+F 0 "H2" H 10250 2853 50  0000 L CNN
+F 1 "MountingHole_Pad" H 10250 2808 50  0001 L CNN
+F 2 "MountingHole:MountingHole_2.7mm_M2.5_Pad_Via" H 10150 2850 50  0001 C CNN
+F 3 "~" H 10150 2850 50  0001 C CNN
+	1    10150 2850
 	1    0    0    -1
 $EndComp
 $Comp
-L Mechanical:MountingHole_Pad H?
+L Mechanical:MountingHole_Pad H1
 U 1 1 62DE5DC9
-P 9900 2800
-F 0 "H?" H 10000 2803 50  0000 L CNN
-F 1 "MountingHole_Pad" H 10000 2758 50  0001 L CNN
-F 2 "MountingHole:MountingHole_2.7mm_M2.5_Pad_Via" H 9900 2800 50  0001 C CNN
-F 3 "~" H 9900 2800 50  0001 C CNN
-	1    9900 2800
+P 9850 2850
+F 0 "H1" H 9950 2853 50  0000 L CNN
+F 1 "MountingHole_Pad" H 9950 2808 50  0001 L CNN
+F 2 "MountingHole:MountingHole_2.7mm_M2.5_Pad_Via" H 9850 2850 50  0001 C CNN
+F 3 "~" H 9850 2850 50  0001 C CNN
+	1    9850 2850
 	1    0    0    -1
 $EndComp
 $Comp
-L power:GND #PWR?
+L power:GND #PWR035
 U 1 1 62DF80EC
-P 9900 3000
-F 0 "#PWR?" H 9900 2750 50  0001 C CNN
-F 1 "GND" H 9905 2827 50  0000 C CNN
-F 2 "" H 9900 3000 50  0001 C CNN
-F 3 "" H 9900 3000 50  0001 C CNN
-	1    9900 3000
+P 9850 3050
+F 0 "#PWR035" H 9850 2800 50  0001 C CNN
+F 1 "GND" H 9855 2877 50  0000 C CNN
+F 2 "" H 9850 3050 50  0001 C CNN
+F 3 "" H 9850 3050 50  0001 C CNN
+	1    9850 3050
 	1    0    0    -1
 $EndComp
 Wire Wire Line
-	9900 2900 9900 2950
+	9850 2950 9850 3000
 Wire Wire Line
-	9900 2950 10200 2950
+	9850 3000 10150 3000
 Wire Wire Line
-	10200 2950 10200 2900
-Connection ~ 9900 2950
+	10150 3000 10150 2950
+Connection ~ 9850 3000
 Wire Wire Line
-	9900 2950 9900 3000
+	9850 3000 9850 3050
 Wire Wire Line
-	10500 2900 10500 2950
+	10450 2950 10450 3000
 Wire Wire Line
-	10500 2950 10200 2950
-Connection ~ 10200 2950
+	10450 3000 10150 3000
+Connection ~ 10150 3000
 Wire Wire Line
-	10800 2900 10800 2950
+	10750 2950 10750 3000
 Wire Wire Line
-	10800 2950 10500 2950
-Connection ~ 10500 2950
+	10750 3000 10450 3000
+Connection ~ 10450 3000
 Wire Notes Line
 	500  2050 11200 2050

Commit message: Routing
Connections:
- net AS7341_EN is gone; now on net 1.15: J5.1
- net AS7341_GPIO is gone; now on net 0.02: J5.2
- net AS7341_INT is gone; now on net 0.29: J5.3
- net 0.13: no longer J4.4
- net 0.15: no longer J4.3
- net 1.10: now also J4.3
- net 1.13: now also J4.4
- no-connect marks 12 -> 7
Changed lines of the file:
@@
 Wire Wire Line
 	7550 1300 7700 1300
-Text Label 2350 2550 2    50   ~ 0
+Text Label 2500 2550 2    50   ~ 0
 RX
-Text Label 2350 2650 2    50   ~ 0
+Text Label 2500 2650 2    50   ~ 0
 TX
 $Comp
@@
 	3650 2850 4000 2850
 Wire Wire Line
-	3750 2950 4000 2950
-Wire Wire Line
-	3750 3050 4000 3050
-Text Label 3750 2950 0    50   ~ 0
-SDA
-Text Label 3750 3050 0    50   ~ 0
-SCL
+	3450 2950 4000 2950
+Wire Wire Line
+	3450 3050 4000 3050
+Text Label 3450 2950 0    50   ~ 0
+STEMMA_SDA
+Text Label 3450 3050 0    50   ~ 0
+STEMMA_SCL
 Wire Wire Line
 	5250 2750 5700 2750
@@
 Wire Wire Line
 	9250 1150 9600 1150
-Wire Wire Line
-	900  2550 1100 2550
-Wire Wire Line
-	900  2650 1100 2650
-Wire Wire Line
-	900  2750 1100 2750
-Wire Wire Line
-	900  2850 1100 2850
-Wire Wire Line
-	900  2950 1100 2950
-Text Label 900  2550 0    50   ~ 0
+Text Label 750  2550 0    50   ~ 0
 1.10
-Text Label 900  2650 0    50   ~ 0
+Text Label 750  2650 0    50   ~ 0
 1.13
-Text Label 900  2750 0    50   ~ 0
+Text Label 750  2750 0    50   ~ 0
 1.15
-Text Label 900  2850 0    50   ~ 0
+Text Label 750  2850 0    50   ~ 0
 0.02
-Text Label 900  2950 0    50   ~ 0
+Text Label 750  2950 0    50   ~ 0
 0.29
-Text Label 900  3050 0    50   ~ 0
+Text Label 750  3050 0    50   ~ 0
 0.31
-Text Label 1700 2550 0    50   ~ 0
+Text Label 1850 2550 0    50   ~ 0
 0.10
-Text Label 1700 2750 0    50   ~ 0
+Text Label 1850 2750 0    50   ~ 0
 1.00
-Text Label 1700 2850 0    50   ~ 0
+Text Label 1850 2850 0    50   ~ 0
 0.24
-Text Label 1700 2950 0    50   ~ 0
+Text Label 1850 2950 0    50   ~ 0
 0.22
-Text Label 1700 3050 0    50   ~ 0
+Text Label 1850 3050 0    50   ~ 0
 0.20
-Text Label 1700 3150 0    50   ~ 0
+Text Label 1850 3150 0    50   ~ 0
 0.17
-Text Label 1700 3250 0    50   ~ 0
+Text Label 1850 3250 0    50   ~ 0
 0.15
-Text Label 1700 3350 0    50   ~ 0
+Text Label 1850 3350 0    50   ~ 0
 0.13
-Text Label 1700 2650 0    50   ~ 0
+Text Label 1850 2650 0    50   ~ 0
 0.09
 Wire Wire Line
-	1700 2550 2350 2550
-Wire Wire Line
-	1700 2650 2350 2650
-Text Label 2350 3250 2    50   ~ 0
+	1850 2550 2500 2550
+Wire Wire Line
+	1850 2650 2500 2650
+Text Label 2500 3250 2    50   ~ 0
 SDA
-Text Label 2350 3350 2    50   ~ 0
+Text Label 2500 3350 2    50   ~ 0
 SCL
 Wire Wire Line
-	1700 3250 2350 3250
-Wire Wire Line
-	1700 3350 2350 3350
-Text Label 2350 3150 2    50   ~ 0
+	1850 3250 2500 3250
+Wire Wire Line
+	1850 3350 2500 3350
+Text Label 2500 3150 2    50   ~ 0
 ADC_DRDY
 Wire Wire Line
-	1700 3150 2350 3150
+	1850 3150 2500 3150
 $Comp
 L SM04B-SRSS-TB_LF__SN_:SM04B-SRSS-TB(LF)(SN) J6
@@
 Text Label 8050 5400 0    50   ~ 0
 LS_A4
-Text Label 2350 2750 2    50   ~ 0
+Text Label 2500 2750 2    50   ~ 0
 LS_A1
-Text Label 2350 2950 2    50   ~ 0
+Text Label 2500 2950 2    50   ~ 0
 LS_A3
-Text Label 2350 2850 2    50   ~ 0
+Text Label 2500 2850 2    50   ~ 0
 LS_A2
-Text Label 2350 3050 2    50   ~ 0
+Text Label 2500 3050 2    50   ~ 0
 LS_A4
 Wire Wire Line
-	1700 2750 2350 2750
-Wire Wire Line
-	1700 2850 2350 2850
-Wire Wire Line
-	1700 2950 2350 2950
-Wire Wire Line
-	1700 3050 2350 3050
+	1850 2750 2500 2750
+Wire Wire Line
+	1850 2850 2500 2850
+Wire Wire Line
+	1850 2950 2500 2950
+Wire Wire Line
+	1850 3050 2500 3050
 Wire Wire Line
 	4900 1800 5450 1800
@@
 BUTTON
 Wire Wire Line
-	900  3050 1500 3050
+	750  3050 1500 3050
 Text Notes 4550 650  0    50   ~ 0
 nRF52840 Dongle
@@
 Text Notes 600  650  0    50   ~ 0
 Power Input
-NoConn ~ 1100 2550
-NoConn ~ 1100 2650
-NoConn ~ 1100 2750
-NoConn ~ 1100 2850
-NoConn ~ 1100 2950
 Wire Notes Line
 	500  3950 11200 3950
@@
 Text Notes 9550 2250 0    50   ~ 0
 Mounting Holes
+Text Label 1500 2750 2    50   ~ 0
+AS7341_EN
+Text Label 1500 2850 2    50   ~ 0
+AS7341_GPIO
+Text Label 1500 2950 2    50   ~ 0
+AS7341_INT
+Wire Wire Line
+	750  2550 1500 2550
+Wire Wire Line
+	750  2650 1500 2650
+Wire Wire Line
+	750  2750 1500 2750
+Wire Wire Line
+	750  2850 1500 2850
+Wire Wire Line
+	750  2950 1500 2950
+Text Label 1500 2550 2    50   ~ 0
+STEMMA_SDA
+Text Label 1500 2650 2    50   ~ 0
+STEMMA_SCL
 $EndSCHEMATC

Commit message: Add C12880MA socket
Parts:
- added IC?: TXU0204PWR, SOP65P640X120-14N, symbol TXU0204PWR:TXU0204PWR
- added J?: C12880MA, Package_DIP:DIP-14_W7.62mm_SMDSocket_SmallPads, symbol Connector_Generic:Conn_02x07_Counter_Clockwise
- added U?: LMV792MM, SOP50P490X110-10N, symbol LMV792MM:LMV792MM
Connections:
- net +5V: now also J?.1 (Pin_1), J?.5 (Pin_5)
- net CLK: now also J?.6 (Pin_6)
- net EOS: now also J?.13 (Pin_13)
- net GND: now also J?.2 (Pin_2), J?.7 (Pin_7)
- net START: now also J?.8 (Pin_8)
- net TRG: now also J?.9 (Pin_9)
- net VIDEO: now also J?.14 (Pin_14)
- no-connect marks 7 -> 12
Other:
- note added: "1"
- note added: "10"
- note added: "2"
- note added: "3"
- note added: "4"
- note added: "5"
- note added: "6"
- note added: "7"
- note added: "8"
- note added: "9"
- moved on the sheet: C6, C7, J8, U3

Commit message: Change level-shifter to TXU0204
Parts:
- removed U3: LSF0204DPWR, SOP65P640X120-14N, symbol LSF0204DPWR:LSF0204DPWR
- added R? (x3): 10k, Resistor_SMD:R_0603_1608Metric, symbol Device:R_Small
- added U? (x3): Opamp_Dual, LMV792MM:SOP50P490X110-10N, symbol LMV792MM:Opamp_Dual
Connections:
- net +5V: now also IC?.14 (VCCB), IC?.8 (OE), U?.10 (V+), U?.5 (ENA), U?.6 (ENB); no longer U1.12 (AVDD)
- net 0.13: no longer U1.16 (SCL)
- net 0.15: no longer U1.15 (SDA)
- net 0.17: now also U?.8 (INB-), U?.9 (OUTB); no longer U1.14 (~DRDY)
- net 0.20: now also IC?.5 (A4Y)
- net 0.22: now also IC?.4 (A3Y)
- net 0.24: now also IC?.3 (A2)
- net 1.00: now also IC?.2 (A1)
- net CLK: now also IC?.13 (B1Y)
- net EOS: now also IC?.10 (B4)
- net GND: now also IC?.7 (GND), U?.4 (V-), R?.2, R?.2; no longer U1.4 (DGND), U1.5 (AGND)
- net START: now also IC?.12 (B2Y)
- net TRG: now also IC?.11 (B3)
- net VDD: now also IC?.1 (VCCA)
- net VIDEO: now also U?.3 (INA+); no longer U1.11 (AIN0)
- net 5V_FOLLOWER_OUT: now reaches U?.1 (OUTA)
- net 5V_FOLLOWER_OUT: now also U?.2 (INA-), R?.1
- net at U?.7 (INB+): now also R?.1, R?.1, R?.2
- new net ADC_DRDY: U1.14 (~DRDY)
- new net SCL: U1.16 (SCL)
- new net SDA: U1.15 (SDA)
Other:
- note added: "Video Treatment"
- note removed: "Video ADC"
- moved on the sheet: C1, C4, C5, C6, C7, JP1, U1, U?
