File: project-nrf-C12880MA-motherboard.kicad_pcb (KiCad board)
At the start: 2 copper layers, 22 parts, among them J1 Left, J2 Right, J3 PJ-036AH-SMT-TR, J4 SM04B-SRSS-TB(LF)(SN), J5 SM04B-SRSS-TB(LF)(SN), J6 SM04B-SRSS-TB(LF)(SN), J7 1702473, J8 C12880MA Breakboard v2, U1 ADS1219IPWR, U2 TPS7A0350PDBVR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

Commit message: First placement
Parts:
- added H1: MountingHole_Pad, MountingHole:MountingHole_2.7mm_M2.5_Pad_Via, F.Cu at (19.1, 24.1)
- added H2: MountingHole_Pad, MountingHole:MountingHole_2.7mm_M2.5_Pad_Via, F.Cu at (97.8, 24.1)
- added H3: MountingHole_Pad, MountingHole:MountingHole_2.7mm_M2.5_Pad_Via, F.Cu at (19.1, 73.7)
- added H4: MountingHole_Pad, MountingHole:MountingHole_2.7mm_M2.5_Pad_Via, F.Cu at (97.8, 73.7)
- moved S1 139.9 mm to (19.1, 57.1), turned to 270 degrees
- moved R1 119.8 mm to (31.8, 39.4), turned to 90 degrees
- moved C6 101.0 mm to (54.6, 39.4), turned to 180 degrees
- moved C7 92.1 mm to (54.6, 31.8), turned to 180 degrees
- moved D1 87.5 mm to (48.3, 55.9), turned to 270 degrees
- moved C3 86.8 mm to (52.1, 44.5)
- moved C2 81.6 mm to (52.1, 52.1)
- moved U2 80.2 mm to (52.0, 48.2), turned to 90 degrees
- moved C5 75.1 mm to (83.8, 74.9), turned to 270 degrees
- moved C4 74.7 mm to (83.8, 71.1), turned to 90 degrees
- moved C1 60.3 mm to (85.1, 68.6), turned to 180 degrees
- moved J4 49.8 mm to (20.3, 31.8), turned to 270 degrees
- moved J5 49.8 mm to (20.3, 40.6), turned to 270 degrees
- moved J3 28.1 mm to (52.1, 62.2)
- moved JP1 14.5 mm to (80.0, 72.4), turned to 270 degrees
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Other:
- board outline added: 86.4 x 57.1 mm

Commit message: Placement 2
Parts:
- moved JP1 16.9 mm to (96.5, 68.6), turned to 0 degrees
- moved J7 13.3 mm to (19.1, 64.8), turned to 270 degrees
- moved C2 5.46 mm to (48.9, 56.5)
- moved C3 5.46 mm to (48.9, 48.9)
- moved U2 5.46 mm to (48.8, 52.7)
- moved S1 5.08 mm to (19.1, 52.1)
- moved D1 3.86 mm to (52.1, 55.2)
- moved C1 2.01 mm to (83.2, 69.2)
- moved U1 2.01 mm to (87.0, 73.0)
- moved J6 2.01 mm to (51.4, 26.0)
- moved C6 2.01 mm to (55.2, 41.3)
- moved C7 2.01 mm to (55.2, 33.7)
- moved U3 2.01 mm to (54.0, 37.5)
- moved C4 2.01 mm to (81.9, 71.8)
- moved C5 2.01 mm to (81.9, 75.6)
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Other:
- board size 86.4 x 57.1 mm -> 86.4 x 57.2 mm

Commit message: Routing
Parts:
- moved C6 8.01 mm to (51.8, 34.0), turned to 0 degrees
- moved C3 6.98 mm to (54.6, 52.9), turned to 270 degrees
- moved D1 5.17 mm to (47.5, 57.7)
- moved C2 3.73 mm to (48.0, 52.9), turned to 270 degrees
- moved U2 2.64 mm to (51.5, 52.9), turned to 0 degrees
- moved C5 1.92 mm to (82.2, 73.7)
- moved U1 1.30 mm to (87.2, 71.8)
- moved C4 1.30 mm to (82.2, 70.5)
- moved C1 1.20 mm to (83.6, 68.1)
- moved C7 0.97 mm to (56.1, 34.0)
Connections:
- J4 pad 3: /0.15 -> /1.10
- J4 pad 4: /0.13 -> /1.13
- J5 pad 1: /AS7341_EN -> /1.15
- J5 pad 2: /AS7341_GPIO -> /0.02
- J5 pad 3: /AS7341_INT -> /0.29
Routing:
- net VDD: track 0.00 -> 203.7 mm, vias 0 -> 4
- net +5V: track 0.00 -> 83.1 mm
- net /0.17: track 0.00 -> 82.1 mm
- net /0.15: track 0.00 -> 75.8 mm
- net /0.13: track 0.00 -> 63.1 mm
- net GND: track 0.00 -> 50.6 mm, vias 0 -> 207
- net /CLK: track 0.00 -> 44.6 mm
- net /START: track 0.00 -> 39.9 mm
- net /0.31: track 0.00 -> 37.1 mm
- net /TRG: track 0.00 -> 36.2 mm
- net /EOS: track 0.00 -> 33.0 mm
- net /0.10: track 0.00 -> 15.5 mm
- net /0.02: track 0.00 -> 13.6 mm
- net /1.00: track 0.00 -> 13.2 mm
- net /1.13: track 0.00 -> 11.8 mm
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- added copper zone on F.Cu, net +5V
- added copper zone on B.Cu, net GND
- added copper zone on F.Cu, net GND
- added copper zone on F.Cu, net Net-(D1-Pad2)
- added copper zone on F.Cu, net VCC
Other:
- rule via_min_drill: 0.3 -> 0.254
- board text added: "AS7341.IO"
- board text added: "François Gervais 15 avril 2022 v1.0.0"
- board text added: "Stemma.QT"
- board text added: "UART"
- board text added: "nRF52840 Dongle"

Commit message: Placement done
Parts:
- removed C1, C5: 0.1uF, Capacitor_SMD:C_0603_1608Metric
- removed JP1: SolderJumper_3_Bridged12, Jumper:SolderJumper-3_P1.3mm_Bridged12_RoundedPad1.0x1.5mm
- removed U3: LSF0204DPWR, LSF0204DPWR:SOP65P640X120-14N
- added IC1: TXU0204PWR, LSF0204DPWR:SOP65P640X120-14N, F.Cu at (50.8, 34.5)
- added R2: 10k, Resistor_SMD:R_0603_1608Metric, F.Cu at (52.1, 41.4)
- added R3: 10k, Resistor_SMD:R_0603_1608Metric, F.Cu at (48.8, 39.6)
- added R4: 10k, Resistor_SMD:R_0603_1608Metric, F.Cu at (48.8, 41.4)
- J8: value C12880MA Breakboard v2 -> C12880MA; footprint HARTING_15650122601000:15650122601000 -> Package_DIP:DIP-14_W7.62mm_SMDSocket_SmallPads
- U1: value ADS1219IPWR -> Opamp_Dual; footprint ADS1219IPWR:SOP65P640X120-16N -> LMV792MM:SOP50P490X110-10N
- moved J7 51.5 mm to (68.6, 50.8), turned to 90 degrees
- moved U1 46.1 mm to (50.5, 43.9)
- moved C4 41.1 mm to (48.8, 46.5), turned to 0 degrees
- moved J8 32.7 mm to (64.8, 32.5)
- moved H4 30.7 mm to (69.2, 61.6)
- moved C3 21.5 mm to (33.8, 47.5), turned to 0 degrees
- moved U2 17.8 mm to (33.8, 50.6), turned to 90 degrees
- moved C2 14.2 mm to (33.8, 54.1), turned to 0 degrees
- moved H3 12.7 mm to (18.4, 61.6)
- moved J3 12.1 mm to (53.3, 50.8)
- moved D1 11.2 mm to (38.6, 50.8), turned to 0 degrees
- moved H2 9.55 mm to (87.6, 25.4)
- moved C6 4.85 mm to (48.3, 30.7)
- moved C7 4.33 mm to (53.3, 30.7)
Connections:
- net /LED renamed Net-(J8-Pad11)
- J8 pad 1: /3V3 -> +5V
- J8 pad 10: /VIDEO -> Net-(J8-Pad10)
- J8 pad 13: GND -> /EOS
- J8 pad 14: GND -> /VIDEO
- J8 pad 2: +5V -> GND
- J8 pad 3: GND -> Net-(J8-Pad3)
- J8 pad 4: GND -> Net-(J8-Pad4)
- J8 pad 5: Net-(J8-Pad5) -> +5V
- J8 pad 6: /EOS -> /CLK
- J8 pad 7: /TRG -> GND
- J8 pad 9: /CLK -> /TRG
- U1 pad 1: GND -> Net-(R2-Pad1)
- U1 pad 10: Net-(U1-Pad10) -> +5V
- U1 pad 2: /ADC_ADDR1 -> Net-(R2-Pad1)
- U1 pad 3: VDD -> /VIDEO
- U1 pad 5: GND -> +5V
- U1 pad 6: Net-(U1-Pad6) -> +5V
- U1 pad 8: GND -> /0.13
- U1 pad 9: +5V -> /0.13
Routing:
- net VDD: track 203.7 -> 69.3 mm, vias 4 -> 0
- net +5V: track 83.1 -> 0.00 mm
- net /0.17: track 82.1 -> 0.00 mm
- net /0.15: track 75.8 -> 0.00 mm
- net /0.13: track 63.1 -> 0.50 mm
- net /CLK: track 44.6 -> 0.00 mm
- net /0.31: track 37.1 -> 81.2 mm
- net /START: track 39.9 -> 0.00 mm
- net /TRG: track 36.2 -> 0.00 mm
- net /EOS: track 33.0 -> 0.00 mm
- net GND: track 50.6 -> 22.8 mm, vias 207 -> 21
- net /1.00: track 13.2 -> 0.00 mm
- net /0.22: track 11.6 -> 0.00 mm
- net /0.24: track 9.12 -> 0.00 mm
- net /ADC_ADDR1: track 8.98 -> 0.00 mm
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Other:
- board size 86.4 x 57.2 mm -> 58.4 x 44.5 mm
- board text removed: "C12880MA Breakout"

Commit message: Routing done
Parts:
- removed H2: MountingHole_Pad, MountingHole:MountingHole_2.7mm_M2.5_Pad_Via
- moved R1 3.06 mm to (32.0, 42.4), turned to 270 degrees
Connections:
- IC1 pad 12: /START -> /CLK
- IC1 pad 13: /CLK -> /START
- J6 pad 2: /0.10 -> /0.09
- J6 pad 3: /0.09 -> /0.10
- J7 pad 1: /0.31 -> /0.13
- R1 pad 2: /0.31 -> /0.13
- S1 pad 1: /0.31 -> /0.13
- S1 pad 2: /0.31 -> /0.13
- U1 pad 8: /0.13 -> /0.31
- U1 pad 9: /0.13 -> /0.31
Routing:
- net +5V: track 0.00 -> 101.6 mm
- net /0.13: track 0.50 -> 88.3 mm
- net /0.31: track 81.2 -> 23.2 mm
- net GND: track 22.8 -> 45.4 mm, vias 21 -> 137
- net /CLK: track 0.00 -> 20.8 mm
- net /TRG: track 0.00 -> 15.5 mm
- net VDD: track 69.3 -> 82.5 mm
- net /START: track 0.00 -> 13.2 mm
- net /VIDEO: track 0.00 -> 9.84 mm
- net /1.00: track 0.00 -> 8.81 mm
- net /EOS: track 0.00 -> 8.28 mm
- net /0.22: track 0.00 -> 8.09 mm
- net Net-(R2-Pad2): track 0.00 -> 6.51 mm
- net /0.20: track 0.00 -> 6.00 mm
- net /0.24: track 0.00 -> 4.73 mm
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Other:
- board text added: "1"
- board text added: "C12880MA"
- board text added: "François Gervais 23 avril 2022 v"
- board text removed: "François Gervais 15 avril 2022 v1.0.0"
